Commit message: mod for frame fix to world

File: src/atr_rov_description/urdf/atr_rov.urdf.xacro (robot description, xacro)
@@ -25,5 +25,5 @@
       <parent link="world"/>
       <child  link="base_link"/>
-      <origin xyz="0 0 0.175" rpy="3.142 0 0"/>
+      <origin xyz="0 0 0" rpy="0 0 0"/>
     </joint>
   </xacro:if>

Commit message: correct joint direction and gazebo spawn

File: src/atr_rov_description/urdf/atr_rov.urdf.xacro (robot description, xacro)
@@ -19,4 +19,8 @@
   <xacro:property name="com_rpy"
     value="${'3.142 0 0' if '$(arg fixed_to_world)' == 'true' else '0 0 0'}"/>
+  <!-- Tag to find the mesh directory for both display and simulation.
+  The xacro arg allows the path to be overridden if needed, but by default
+  it uses the meshes directory in this package. -->
+  <xacro:arg name="mesh_path" default="package://atr_rov_description/meshes"/>
   <!-- ── World anchor — RViz2 display only ────────────────────── -->
   <xacro:if value="$(arg fixed_to_world)">
@@ -41,5 +45,5 @@
       <origin xyz="0.1975 0.35 0.175" rpy=" 3.142 0 0"/>
       <geometry>
-        <mesh filename="package://atr_rov_description/meshes/4mm_houston_scaled_32mb.stl"
+        <mesh filename="$(arg mesh_path)/4mm_houston_scaled_32mb.stl"
               scale="0.001 0.001 0.001"/>
       </geometry>
@@ -50,7 +54,9 @@
     <collision>
       <origin xyz="0.1975 0.35 0.175" rpy="3.142 0 0"/>
+      <!-- <origin xyz="-0.12 0 0.23" rpy="3.142 0 0"/> -->
       <geometry>
-        <mesh filename="package://atr_rov_description/meshes/4mm_houston_scaled_32mb.stl"
+        <mesh filename="$(arg mesh_path)/4mm_houston_scaled_32mb.stl"
               scale="0.001 0.001 0.001"/>
+        <!-- <box size="1.97 0.6 0.46"/> -->
       </geometry>
     </collision>
@@ -95,51 +101,115 @@
     bridge or flip the rotation by π (add 3.14159 to the relevant angle).
   -->
-  <link name="thruster_1_link"/>
-  <joint name="thruster_1_joint" type="fixed">
+  <link name="thruster_1_link">
+    <inertial>
+      <mass value="0.001"/>
+      <inertia ixx="0.000001" ixy="0" ixz="0"
+              iyy="0.000001" iyz="0" izz="0.000001"/>
+    </inertial>
+  </link>
+  <joint name="thruster_1_joint" type="revolute">
     <parent link="base_link"/>
     <child  link="thruster_1_link"/>
     <origin xyz="0.371365 -0.15363 0.09" rpy="0 0 0"/>
-  </joint>
-  <link name="thruster_2_link"/>
-  <joint name="thruster_2_joint" type="fixed">
+    <axis xyz="0 0 1"/>
+    <limit lower="-1e9" upper="1e9" effort="100" velocity="1000"/>
+  </joint>
+  <link name="thruster_2_link">
+    <inertial>
+      <mass value="0.001"/>
+      <inertia ixx="0.000001" ixy="0" ixz="0"
+              iyy="0.000001" iyz="0" izz="0.000001"/>
+    </inertial>
+  </link>
+  <joint name="thruster_2_joint" type="revolute">
     <parent link="base_link"/>
     <child  link="thruster_2_link"/>
     <origin xyz="0.371365 0.14037 0.09" rpy="0 0 0"/>
-  </joint>
-  <link name="thruster_3_link"/>
-  <joint name="thruster_3_joint" type="fixed">
+    <axis xyz="0 0 1"/>
+    <limit lower="-1e9" upper="1e9" effort="100" velocity="1000"/>
+  </joint>
+  <link name="thruster_3_link">
+    <inertial>
+      <mass value="0.001"/>
+      <inertia ixx="0.000001" ixy="0" ixz="0"
+              iyy="0.000001" iyz="0" izz="0.000001"/>
+    </inertial>
+  </link>
+  <joint name="thruster_3_joint" type="revolute">
     <parent link="base_link"/>
     <child  link="thruster_3_link"/>
     <origin xyz="-0.514 0.14037 0.09" rpy="0 0 0"/>
-  </joint>
-  <link name="thruster_4_link"/>
-  <joint name="thruster_4_joint" type="fixed">
+    <axis xyz="0 0 1"/>
+    <limit lower="-1e9" upper="1e9" effort="100" velocity="1000"/>
+  </joint>
+  <link name="thruster_4_link">
+    <inertial>
+      <mass value="0.001"/>
+      <inertia ixx="0.000001" ixy="0" ixz="0"
+              iyy="0.000001" iyz="0" izz="0.000001"/>
+    </inertial>
+  </link>
+  <joint name="thruster_4_joint" type="revolute">
     <parent link="base_link"/>
     <child  link="thruster_4_link"/>
     <origin xyz="-0.514 -0.15363 0.09" rpy="0 0 0"/>
-  </joint>
-  <link name="thruster_5_link"/>
-  <joint name="thruster_5_joint" type="fixed">
+    <axis xyz="0 0 1"/>
+    <limit lower="-1e9" upper="1e9" effort="100" velocity="1000"/>
+  </joint>
+  <link name="thruster_5_link">
+    <inertial>
+      <mass value="0.001"/>
+      <inertia ixx="0.000001" ixy="0" ixz="0"
+              iyy="0.000001" iyz="0" izz="0.000001"/>
+    </inertial>
+  </link>
+  <joint name="thruster_5_joint" type="revolute">
     <parent link="base_link"/>
     <child  link="thruster_5_link"/>
     <origin xyz="0.11 -0.148 0.32" rpy="0 0 0"/>
-  </joint>
-  <link name="thruster_6_link"/>
-  <joint name="thruster_6_joint" type="fixed">
+    <axis xyz="1 0 0"/>
+    <limit lower="-1e9" upper="1e9" effort="100" velocity="1000"/>
+  </joint>
+  <link name="thruster_6_link">
+    <inertial>
+      <mass value="0.001"/>
+      <inertia ixx="0.000001" ixy="0" ixz="0"
+              iyy="0.000001" iyz="0" izz="0.000001"/>
+    </inertial>
+  </link>
+  <joint name="thruster_6_joint" type="revolute">
     <parent link="base_link"/>
     <child  link="thruster_6_link"/>
     <origin xyz="0.11 0.13 0.32" rpy="0 0 0"/>
-  </joint>
-  <link name="thruster_7_link"/>
-  <joint name="thruster_7_joint" type="fixed">
+    <axis xyz="1 0 0"/>
+    <limit lower="-1e9" upper="1e9" effort="100" velocity="1000"/>
+  </joint>
+  <link name="thruster_7_link">
+    <inertial>
+      <mass value="0.001"/>
+      <inertia ixx="0.000001" ixy="0" ixz="0"
+              iyy="0.000001" iyz="0" izz="0.000001"/>
+    </inertial>
+  </link>
+  <joint name="thruster_7_joint" type="revolute">
     <parent link="base_link"/>
     <child  link="thruster_7_link"/>
     <origin xyz="-0.36 0.075 0.379" rpy="0 0 0"/>
-  </joint>
-  <link name="thruster_8_link"/>
-  <joint name="thruster_8_joint" type="fixed">
+    <axis xyz="0 1 0"/>
+    <limit lower="-1e9" upper="1e9" effort="100" velocity="1000"/>
+  </joint>
+  <link name="thruster_8_link">
+    <inertial>
+      <mass value="0.001"/>
+      <inertia ixx="0.000001" ixy="0" ixz="0"
+              iyy="0.000001" iyz="0" izz="0.000001"/>
+    </inertial>
+  </link>
+  <joint name="thruster_8_joint" type="revolute">
     <parent link="base_link"/>
     <child  link="thruster_8_link"/>
     <origin xyz="0.215 0.075 0.379" rpy="0 0 0"/>
+    <axis xyz="0 1 0"/>
+    <limit lower="-1e9" upper="1e9" effort="100" velocity="1000"/>
   </joint>
   <!-- ── Gazebo Fortress — Hydrodynamics plugin ────────────────── -->
@@ -171,15 +241,9 @@
     </plugin>
   </gazebo>
-  <!-- ── Gazebo Fortress — Buoyancy plugin ─────────────────────── -->
-  <gazebo>
-    <plugin filename="ignition-gazebo-buoyancy-system"
-            name="ignition::gazebo::systems::Buoyancy">
-      <uniform_fluid_density>1000</uniform_fluid_density>
-    </plugin>
-  </gazebo>
   <!-- ── Gazebo Fortress — Thruster plugins (T1–T8) ────────────── -->
   <gazebo>
-    <plugin filename="ignition-gazebo-thruster-system"
-            name="ignition::gazebo::systems::Thruster">
+    <plugin
+      filename="ignition-gazebo-thruster-system"
+      name="ignition::gazebo::systems::Thruster">
       <namespace>atr_mp_rov</namespace>
       <joint_name>thruster_1_joint</joint_name>
@@ -188,6 +252,8 @@
       <propeller_diameter>0.1</propeller_diameter>
       <velocity_control>true</velocity_control>
-      <topic>/atr_mp_rov/thrusters/1/force</topic>
-    </plugin>
+      <topic>thrusters/1/force</topic>
+    </plugin>
+  </gazebo>
+  <gazebo>
     <plugin filename="ignition-gazebo-thruster-system"
             name="ignition::gazebo::systems::Thruster">
@@ -198,6 +264,8 @@
       <propeller_diameter>0.1</propeller_diameter>
       <velocity_control>true</velocity_control>
-      <topic>/atr_mp_rov/thrusters/2/force</topic>
-    </plugin>
+      <topic>thrusters/2/force</topic>
+    </plugin>
+  </gazebo>
+  <gazebo>
     <plugin filename="ignition-gazebo-thruster-system"
             name="ignition::gazebo::systems::Thruster">
@@ -208,6 +276,8 @@
       <propeller_diameter>0.1</propeller_diameter>
       <velocity_control>true</velocity_control>
-      <topic>/atr_mp_rov/thrusters/3/force</topic>
-    </plugin>
+      <topic>thrusters/3/force</topic>
+    </plugin>
+  </gazebo>
+  <gazebo>
     <plugin filename="ignition-gazebo-thruster-system"
             name="ignition::gazebo::systems::Thruster">
@@ -218,6 +288,8 @@
       <propeller_diameter>0.1</propeller_diameter>
       <velocity_control>true</velocity_control>
-      <topic>/atr_mp_rov/thrusters/4/force</topic>
-    </plugin>
+      <topic>thrusters/4/force</topic>
+    </plugin>
+  </gazebo>
+  <gazebo>
     <plugin filename="ignition-gazebo-thruster-system"
             name="ignition::gazebo::systems::Thruster">
@@ -228,6 +300,8 @@
       <propeller_diameter>0.1</propeller_diameter>
       <velocity_control>true</velocity_control>
-      <topic>/atr_mp_rov/thrusters/5/force</topic>
-    </plugin>
+      <topic>thrusters/5/force</topic>
+    </plugin>
+  </gazebo>
+  <gazebo>
     <plugin filename="ignition-gazebo-thruster-system"
             name="ignition::gazebo::systems::Thruster">
@@ -238,6 +312,8 @@
       <propeller_diameter>0.1</propeller_diameter>
       <velocity_control>true</velocity_control>
-      <topic>/atr_mp_rov/thrusters/6/force</topic>
-    </plugin>
+      <topic>thrusters/6/force</topic>
+    </plugin>
+  </gazebo>
+  <gazebo>
     <plugin filename="ignition-gazebo-thruster-system"
             name="ignition::gazebo::systems::Thruster">
@@ -248,6 +324,8 @@
       <propeller_diameter>0.1</propeller_diameter>
       <velocity_control>true</velocity_control>
-      <topic>/atr_mp_rov/thrusters/7/force</topic>
-    </plugin>
+      <topic>thrusters/7/force</topic>
+    </plugin>
+  </gazebo>
+  <gazebo>
     <plugin filename="ignition-gazebo-thruster-system"
             name="ignition::gazebo::systems::Thruster">
@@ -258,5 +336,5 @@
       <propeller_diameter>0.1</propeller_diameter>
       <velocity_control>true</velocity_control>
-      <topic>/atr_mp_rov/thrusters/8/force</topic>
+      <topic>thrusters/8/force</topic>
     </plugin>
   </gazebo>
@@ -289,6 +367,6 @@
         </linear_acceleration>
       </imu>
-      <plugin filename="ignition-gazebo-imu-system"
-              name="ignition::gazebo::systems::Imu"/>
+      <!-- <plugin filename="ignition-gazebo-imu-system"
+              name="ignition::gazebo::systems::Imu"/> -->
     </sensor>
   </gazebo>
@@ -303,6 +381,6 @@
         </pressure>
       </air_pressure>
-      <plugin filename="ignition-gazebo-air-pressure-system"
-              name="ignition::gazebo::systems::AirPressure"/>
+      <!-- <plugin filename="ignition-gazebo-air-pressure-system"
+              name="ignition::gazebo::systems::AirPressure"/> -->
     </sensor>
   </gazebo>

Commit message: facing physics rate issue

File: src/atr_rov_description/urdf/atr_rov.urdf.xacro (robot description, xacro)
@@ -35,5 +35,5 @@
     <inertial>
       <!-- CoM offset — switches between display and physics frame -->
-      <origin xyz="0.06136 -0.00281 ${com_z}" rpy="${com_rpy}"/>
+      <origin xyz="0.06136 -0.00281 ${com_z}" rpy="0 0 0"/>
       <mass value="${mass}"/>
       <inertia ixx="${ixx}" ixy="${ixy}" ixz="${ixz}"
@@ -45,5 +45,5 @@
       <origin xyz="0.1975 0.35 0.175" rpy=" 3.142 0 0"/>
       <geometry>
-        <mesh filename="$(arg mesh_path)/4mm_houston_scaled_32mb.stl"
+        <mesh filename="$(arg mesh_path)/4mm_houston_scaled_16mb.stl"
               scale="0.001 0.001 0.001"/>
       </geometry>
@@ -54,9 +54,7 @@
     <collision>
       <origin xyz="0.1975 0.35 0.175" rpy="3.142 0 0"/>
-      <!-- <origin xyz="-0.12 0 0.23" rpy="3.142 0 0"/> -->
       <geometry>
-        <mesh filename="$(arg mesh_path)/4mm_houston_scaled_32mb.stl"
+        <mesh filename="$(arg mesh_path)/4mm_houston_scaled_16mb.stl"
               scale="0.001 0.001 0.001"/>
-        <!-- <box size="1.97 0.6 0.46"/> -->
       </geometry>
     </collision>
@@ -108,10 +106,10 @@
     </inertial>
   </link>
-  <joint name="thruster_1_joint" type="revolute">
+  <joint name="thruster_1_joint" type="continuous">
     <parent link="base_link"/>
     <child  link="thruster_1_link"/>
     <origin xyz="0.371365 -0.15363 0.09" rpy="0 0 0"/>
     <axis xyz="0 0 1"/>
-    <limit lower="-1e9" upper="1e9" effort="100" velocity="1000"/>
+    <!-- <limit lower="-1e9" upper="1e9" effort="100" velocity="1000"/> -->
   </joint>
   <link name="thruster_2_link">
@@ -122,10 +120,10 @@
     </inertial>
   </link>
-  <joint name="thruster_2_joint" type="revolute">
+  <joint name="thruster_2_joint" type="continuous">
     <parent link="base_link"/>
     <child  link="thruster_2_link"/>
     <origin xyz="0.371365 0.14037 0.09" rpy="0 0 0"/>
     <axis xyz="0 0 1"/>
-    <limit lower="-1e9" upper="1e9" effort="100" velocity="1000"/>
+    <!-- <limit lower="-1e9" upper="1e9" effort="100" velocity="1000"/> -->
   </joint>
   <link name="thruster_3_link">
@@ -136,10 +134,10 @@
     </inertial>
   </link>
-  <joint name="thruster_3_joint" type="revolute">
+  <joint name="thruster_3_joint" type="continuous">
     <parent link="base_link"/>
     <child  link="thruster_3_link"/>
     <origin xyz="-0.514 0.14037 0.09" rpy="0 0 0"/>
     <axis xyz="0 0 1"/>
-    <limit lower="-1e9" upper="1e9" effort="100" velocity="1000"/>
+    <!-- <limit lower="-1e9" upper="1e9" effort="100" velocity="1000"/> -->
   </joint>
   <link name="thruster_4_link">
@@ -150,10 +148,10 @@
     </inertial>
   </link>
-  <joint name="thruster_4_joint" type="revolute">
+  <joint name="thruster_4_joint" type="continuous">
     <parent link="base_link"/>
     <child  link="thruster_4_link"/>
     <origin xyz="-0.514 -0.15363 0.09" rpy="0 0 0"/>
     <axis xyz="0 0 1"/>
-    <limit lower="-1e9" upper="1e9" effort="100" velocity="1000"/>
+    <!-- <limit lower="-1e9" upper="1e9" effort="100" velocity="1000"/> -->
   </joint>
   <link name="thruster_5_link">
@@ -164,10 +162,10 @@
     </inertial>
   </link>
-  <joint name="thruster_5_joint" type="revolute">
+  <joint name="thruster_5_joint" type="continuous">
     <parent link="base_link"/>
     <child  link="thruster_5_link"/>
     <origin xyz="0.11 -0.148 0.32" rpy="0 0 0"/>
     <axis xyz="1 0 0"/>
-    <limit lower="-1e9" upper="1e9" effort="100" velocity="1000"/>
+    <!-- <limit lower="-1e9" upper="1e9" effort="100" velocity="1000"/> -->
   </joint>
   <link name="thruster_6_link">
@@ -178,10 +176,10 @@
     </inertial>
   </link>
-  <joint name="thruster_6_joint" type="revolute">
+  <joint name="thruster_6_joint" type="continuous">
     <parent link="base_link"/>
     <child  link="thruster_6_link"/>
     <origin xyz="0.11 0.13 0.32" rpy="0 0 0"/>
     <axis xyz="1 0 0"/>
-    <limit lower="-1e9" upper="1e9" effort="100" velocity="1000"/>
+    <!-- <limit lower="-1e9" upper="1e9" effort="100" velocity="1000"/> -->
   </joint>
   <link name="thruster_7_link">
@@ -192,10 +190,10 @@
     </inertial>
   </link>
-  <joint name="thruster_7_joint" type="revolute">
+  <joint name="thruster_7_joint" type="continuous">
     <parent link="base_link"/>
     <child  link="thruster_7_link"/>
     <origin xyz="-0.36 0.075 0.379" rpy="0 0 0"/>
     <axis xyz="0 1 0"/>
-    <limit lower="-1e9" upper="1e9" effort="100" velocity="1000"/>
+    <!-- <limit lower="-1e9" upper="1e9" effort="100" velocity="1000"/> -->
   </joint>
   <link name="thruster_8_link">
@@ -206,10 +204,10 @@
     </inertial>
   </link>
-  <joint name="thruster_8_joint" type="revolute">
+  <joint name="thruster_8_joint" type="continuous">
     <parent link="base_link"/>
     <child  link="thruster_8_link"/>
     <origin xyz="0.215 0.075 0.379" rpy="0 0 0"/>
     <axis xyz="0 1 0"/>
-    <limit lower="-1e9" upper="1e9" effort="100" velocity="1000"/>
+    <!-- <limit lower="-1e9" upper="1e9" effort="100" velocity="1000"/> -->
   </joint>
   <!-- ── Gazebo Fortress — Hydrodynamics plugin ────────────────── -->
@@ -347,5 +345,5 @@
       <robot_base_frame>base_link</robot_base_frame>
       <odom_frame>odom</odom_frame>
-      <publish_rate>100</publish_rate>
+      <publish_rate>50</publish_rate>
     </plugin>
   </gazebo>
@@ -354,5 +352,5 @@
     <sensor name="ins_imu" type="imu">
       <always_on>true</always_on>
-      <update_rate>100</update_rate>
+      <update_rate>50</update_rate>
       <imu>
         <angular_velocity>
@@ -367,6 +365,6 @@
         </linear_acceleration>
       </imu>
-      <!-- <plugin filename="ignition-gazebo-imu-system"
-              name="ignition::gazebo::systems::Imu"/> -->
+      <plugin filename="ignition-gazebo-imu-system"
+              name="ignition::gazebo::systems::Imu"/>
     </sensor>
   </gazebo>

Commit message: stable bot descent

File: src/atr_rov_description/urdf/atr_rov.urdf.xacro (robot description, xacro)
@@ -35,5 +35,5 @@
     <inertial>
       <!-- CoM offset — switches between display and physics frame -->
-      <origin xyz="0.06136 -0.00281 ${com_z}" rpy="0 0 0"/>
+      <origin xyz="-0.11 -0.001 ${com_z}" rpy="0 0 0"/>
       <mass value="${mass}"/>
       <inertia ixx="${ixx}" ixy="${ixy}" ixz="${ixz}"
@@ -53,8 +53,7 @@
     </visual>
     <collision>
-      <origin xyz="0.1975 0.35 0.175" rpy="3.142 0 0"/>
+      <origin xyz="-0.11 -0.001 0.22" rpy=" 0 0 0"/>
       <geometry>
-        <mesh filename="$(arg mesh_path)/4mm_houston_scaled_16mb.stl"
-              scale="0.001 0.001 0.001"/>
+        <box size="1.97 0.6 0.1038"/>
       </geometry>
     </collision>
@@ -101,7 +100,7 @@
   <link name="thruster_1_link">
     <inertial>
-      <mass value="0.001"/>
-      <inertia ixx="0.000001" ixy="0" ixz="0"
-              iyy="0.000001" iyz="0" izz="0.000001"/>
+      <mass value="0.5"/>
+      <inertia ixx="0.001" ixy="0" ixz="0"
+              iyy="0.001" iyz="0" izz="0.001"/>
     </inertial>
   </link>
@@ -115,7 +114,7 @@
   <link name="thruster_2_link">
     <inertial>
-      <mass value="0.001"/>
-      <inertia ixx="0.000001" ixy="0" ixz="0"
-              iyy="0.000001" iyz="0" izz="0.000001"/>
+      <mass value="0.5"/>
+      <inertia ixx="0.001" ixy="0" ixz="0"
+              iyy="0.001" iyz="0" izz="0.001"/>
     </inertial>
   </link>
@@ -129,7 +128,7 @@
   <link name="thruster_3_link">
     <inertial>
-      <mass value="0.001"/>
-      <inertia ixx="0.000001" ixy="0" ixz="0"
-              iyy="0.000001" iyz="0" izz="0.000001"/>
+      <mass value="0.5"/>
+      <inertia ixx="0.001" ixy="0" ixz="0"
+              iyy="0.001" iyz="0" izz="0.001"/>
     </inertial>
   </link>
@@ -143,7 +142,7 @@
   <link name="thruster_4_link">
     <inertial>
-      <mass value="0.001"/>
-      <inertia ixx="0.000001" ixy="0" ixz="0"
-              iyy="0.000001" iyz="0" izz="0.000001"/>
+      <mass value="0.5"/>
+      <inertia ixx="0.001" ixy="0" ixz="0"
+              iyy="0.001" iyz="0" izz="0.001"/>
     </inertial>
   </link>
@@ -157,7 +156,7 @@
   <link name="thruster_5_link">
     <inertial>
-      <mass value="0.001"/>
-      <inertia ixx="0.000001" ixy="0" ixz="0"
-              iyy="0.000001" iyz="0" izz="0.000001"/>
+      <mass value="0.5"/>
+      <inertia ixx="0.001" ixy="0" ixz="0"
+              iyy="0.001" iyz="0" izz="0.001"/>
     </inertial>
   </link>
@@ -171,7 +170,7 @@
   <link name="thruster_6_link">
     <inertial>
-      <mass value="0.001"/>
-      <inertia ixx="0.000001" ixy="0" ixz="0"
-              iyy="0.000001" iyz="0" izz="0.000001"/>
+      <mass value="0.5"/>
+      <inertia ixx="0.001" ixy="0" ixz="0"
+              iyy="0.001" iyz="0" izz="0.001"/>
     </inertial>
   </link>
@@ -185,7 +184,7 @@
   <link name="thruster_7_link">
     <inertial>
-      <mass value="0.001"/>
-      <inertia ixx="0.000001" ixy="0" ixz="0"
-              iyy="0.000001" iyz="0" izz="0.000001"/>
+      <mass value="0.5"/>
+      <inertia ixx="0.001" ixy="0" ixz="0"
+              iyy="0.001" iyz="0" izz="0.001"/>
     </inertial>
   </link>
@@ -199,7 +198,7 @@
   <link name="thruster_8_link">
     <inertial>
-      <mass value="0.001"/>
-      <inertia ixx="0.000001" ixy="0" ixz="0"
-              iyy="0.000001" iyz="0" izz="0.000001"/>
+      <mass value="0.5"/>
+      <inertia ixx="0.001" ixy="0" ixz="0"
+              iyy="0.001" iyz="0" izz="0.001"/>
     </inertial>
   </link>
@@ -217,7 +216,11 @@
       <link_name>base_link</link_name>
       <!-- Added mass (Phase 1 Section 5.1) -->
+      <!-- yDotV/zDotW capped below vehicle mass (119 kg): Ignition applies added
+           mass as an explicit force; M_A > m causes acceleration divergence. -->
+      <!-- <yDotV>-160.95</yDotV> -->
+      <!-- <zDotW>-160.95</zDotW> -->
       <xDotU>-53.65</xDotU>
-      <yDotV>-160.95</yDotV>
-      <zDotW>-160.95</zDotW>
+        <yDotV>-95.0</yDotV>
+        <zDotW>-95.0</zDotW>
       <kDotP>-0.005</kDotP>
       <mDotQ>-1.0</mDotQ>
@@ -236,5 +239,5 @@
       <kPabsP>0.0</kPabsP>
       <mQabsQ>0.0</mQabsQ>
-      <nRabsN>0.0</nRabsN>
+      <nRabsR>0.0</nRabsR>
     </plugin>
   </gazebo>
