Commit message: phase 2 complete

File: src/atr_rov_description/urdf/atr_rov.urdf.xacro (robot description, xacro)
@@ -105,10 +105,10 @@
     </inertial>
   </link>
-  <joint name="thruster_1_joint" type="continuous">
+  <joint name="thruster_1_joint" type="revolute">
     <parent link="base_link"/>
     <child  link="thruster_1_link"/>
     <origin xyz="0.371365 -0.15363 0.09" rpy="0 0 0"/>
     <axis xyz="0 0 1"/>
-    <!-- <limit lower="-1e9" upper="1e9" effort="100" velocity="1000"/> -->
+    <limit lower="-1e6" upper="1e6" effort="1000" velocity="1000"/>
   </joint>
   <link name="thruster_2_link">
@@ -119,10 +119,10 @@
     </inertial>
   </link>
-  <joint name="thruster_2_joint" type="continuous">
+  <joint name="thruster_2_joint" type="revolute">
     <parent link="base_link"/>
     <child  link="thruster_2_link"/>
     <origin xyz="0.371365 0.14037 0.09" rpy="0 0 0"/>
     <axis xyz="0 0 1"/>
-    <!-- <limit lower="-1e9" upper="1e9" effort="100" velocity="1000"/> -->
+    <limit lower="-1e6" upper="1e6" effort="1000" velocity="1000"/>
   </joint>
   <link name="thruster_3_link">
@@ -133,10 +133,10 @@
     </inertial>
   </link>
-  <joint name="thruster_3_joint" type="continuous">
+  <joint name="thruster_3_joint" type="revolute">
     <parent link="base_link"/>
     <child  link="thruster_3_link"/>
     <origin xyz="-0.514 0.14037 0.09" rpy="0 0 0"/>
     <axis xyz="0 0 1"/>
-    <!-- <limit lower="-1e9" upper="1e9" effort="100" velocity="1000"/> -->
+    <limit lower="-1e6" upper="1e6" effort="1000" velocity="1000"/>
   </joint>
   <link name="thruster_4_link">
@@ -147,10 +147,10 @@
     </inertial>
   </link>
-  <joint name="thruster_4_joint" type="continuous">
+  <joint name="thruster_4_joint" type="revolute">
     <parent link="base_link"/>
     <child  link="thruster_4_link"/>
     <origin xyz="-0.514 -0.15363 0.09" rpy="0 0 0"/>
     <axis xyz="0 0 1"/>
-    <!-- <limit lower="-1e9" upper="1e9" effort="100" velocity="1000"/> -->
+    <limit lower="-1e6" upper="1e6" effort="1000" velocity="1000"/>
   </joint>
   <link name="thruster_5_link">
@@ -161,10 +161,10 @@
     </inertial>
   </link>
-  <joint name="thruster_5_joint" type="continuous">
+  <joint name="thruster_5_joint" type="revolute">
     <parent link="base_link"/>
     <child  link="thruster_5_link"/>
     <origin xyz="0.11 -0.148 0.32" rpy="0 0 0"/>
     <axis xyz="1 0 0"/>
-    <!-- <limit lower="-1e9" upper="1e9" effort="100" velocity="1000"/> -->
+    <limit lower="-1e6" upper="1e6" effort="1000" velocity="1000"/>
   </joint>
   <link name="thruster_6_link">
@@ -175,10 +175,10 @@
     </inertial>
   </link>
-  <joint name="thruster_6_joint" type="continuous">
+  <joint name="thruster_6_joint" type="revolute">
     <parent link="base_link"/>
     <child  link="thruster_6_link"/>
     <origin xyz="0.11 0.13 0.32" rpy="0 0 0"/>
     <axis xyz="1 0 0"/>
-    <!-- <limit lower="-1e9" upper="1e9" effort="100" velocity="1000"/> -->
+    <limit lower="-1e6" upper="1e6" effort="1000" velocity="1000"/>
   </joint>
   <link name="thruster_7_link">
@@ -189,10 +189,10 @@
     </inertial>
   </link>
-  <joint name="thruster_7_joint" type="continuous">
+  <joint name="thruster_7_joint" type="revolute">
     <parent link="base_link"/>
     <child  link="thruster_7_link"/>
     <origin xyz="-0.36 0.075 0.379" rpy="0 0 0"/>
     <axis xyz="0 1 0"/>
-    <!-- <limit lower="-1e9" upper="1e9" effort="100" velocity="1000"/> -->
+    <limit lower="-1e6" upper="1e6" effort="1000" velocity="1000"/>
   </joint>
   <link name="thruster_8_link">
@@ -203,10 +203,10 @@
     </inertial>
   </link>
-  <joint name="thruster_8_joint" type="continuous">
+  <joint name="thruster_8_joint" type="revolute">
     <parent link="base_link"/>
     <child  link="thruster_8_link"/>
     <origin xyz="0.215 0.075 0.379" rpy="0 0 0"/>
     <axis xyz="0 1 0"/>
-    <!-- <limit lower="-1e9" upper="1e9" effort="100" velocity="1000"/> -->
+    <limit lower="-1e6" upper="1e6" effort="1000" velocity="1000"/>
   </joint>
   <!-- ── Gazebo Fortress — Hydrodynamics plugin ────────────────── -->
@@ -221,6 +221,6 @@
       <!-- <zDotW>-160.95</zDotW> -->
       <xDotU>-53.65</xDotU>
-        <yDotV>-95.0</yDotV>
-        <zDotW>-95.0</zDotW>
+      <yDotV>-95.0</yDotV>
+      <zDotW>-95.0</zDotW>
       <kDotP>-0.005</kDotP>
       <mDotQ>-1.0</mDotQ>
@@ -242,4 +242,10 @@
     </plugin>
   </gazebo>
+  <!-- Gazebo joint state publisher -->
+  <gazebo>
+    <plugin filename="ignition-gazebo-joint-state-publisher-system"
+            name="ignition::gazebo::systems::JointStatePublisher">
+    </plugin>
+  </gazebo>
   <!-- ── Gazebo Fortress — Thruster plugins (T1–T8) ────────────── -->
   <gazebo>
@@ -252,6 +258,7 @@
       <fluid_density>1000</fluid_density>
       <propeller_diameter>0.1</propeller_diameter>
-      <velocity_control>true</velocity_control>
-      <topic>thrusters/1/force</topic>
+      <!-- <velocity_control>true</velocity_control> -->
+      <!-- <use_angvel_cmd>true</use_angvel_cmd> -->
+      <topic>thrusters/t1/force</topic>
     </plugin>
   </gazebo>
@@ -264,6 +271,7 @@
       <fluid_density>1000</fluid_density>
       <propeller_diameter>0.1</propeller_diameter>
-      <velocity_control>true</velocity_control>
-      <topic>thrusters/2/force</topic>
+      <!-- <velocity_control>true</velocity_control> -->
+      <!-- <use_angvel_cmd>true</use_angvel_cmd> -->
+      <topic>thrusters/t2/force</topic>
     </plugin>
   </gazebo>
@@ -276,6 +284,7 @@
       <fluid_density>1000</fluid_density>
       <propeller_diameter>0.1</propeller_diameter>
-      <velocity_control>true</velocity_control>
-      <topic>thrusters/3/force</topic>
+      <!-- <velocity_control>true</velocity_control> -->
+      <!-- <use_angvel_cmd>true</use_angvel_cmd> -->
+      <topic>thrusters/t3/force</topic>
     </plugin>
   </gazebo>
@@ -288,6 +297,7 @@
       <fluid_density>1000</fluid_density>
       <propeller_diameter>0.1</propeller_diameter>
-      <velocity_control>true</velocity_control>
-      <topic>thrusters/4/force</topic>
+      <!-- <velocity_control>true</velocity_control> -->
+      <!-- <use_angvel_cmd>true</use_angvel_cmd> -->
+      <topic>thrusters/t4/force</topic>
     </plugin>
   </gazebo>
@@ -300,6 +310,7 @@
       <fluid_density>1000</fluid_density>
       <propeller_diameter>0.1</propeller_diameter>
-      <velocity_control>true</velocity_control>
-      <topic>thrusters/5/force</topic>
+      <!-- <velocity_control>true</velocity_control> -->
+      <!-- <use_angvel_cmd>true</use_angvel_cmd> -->
+      <topic>thrusters/t5/force</topic>
     </plugin>
   </gazebo>
@@ -312,6 +323,7 @@
       <fluid_density>1000</fluid_density>
       <propeller_diameter>0.1</propeller_diameter>
-      <velocity_control>true</velocity_control>
-      <topic>thrusters/6/force</topic>
+      <!-- <velocity_control>true</velocity_control> -->
+      <!-- <use_angvel_cmd>true</use_angvel_cmd> -->
+      <topic>thrusters/t6/force</topic>
     </plugin>
   </gazebo>
@@ -324,6 +336,7 @@
       <fluid_density>1000</fluid_density>
       <propeller_diameter>0.1</propeller_diameter>
-      <velocity_control>true</velocity_control>
-      <topic>thrusters/7/force</topic>
+      <!-- <velocity_control>true</velocity_control> -->
+      <!-- <use_angvel_cmd>true</use_angvel_cmd> -->
+      <topic>thrusters/t7/force</topic>
     </plugin>
   </gazebo>
@@ -336,6 +349,7 @@
       <fluid_density>1000</fluid_density>
       <propeller_diameter>0.1</propeller_diameter>
-      <velocity_control>true</velocity_control>
-      <topic>thrusters/8/force</topic>
+      <!-- <velocity_control>true</velocity_control> -->
+      <!-- <use_angvel_cmd>true</use_angvel_cmd> -->
+      <topic>thrusters/t8/force</topic>
     </plugin>
   </gazebo>
@@ -348,5 +362,6 @@
       <robot_base_frame>base_link</robot_base_frame>
       <odom_frame>odom</odom_frame>
-      <publish_rate>50</publish_rate>
+      <publish_rate>100</publish_rate>
+      <dimensions>3</dimensions>
     </plugin>
   </gazebo>
@@ -355,5 +370,5 @@
     <sensor name="ins_imu" type="imu">
       <always_on>true</always_on>
-      <update_rate>50</update_rate>
+      <update_rate>100</update_rate>
       <imu>
         <angular_velocity>
@@ -376,5 +391,5 @@
     <sensor name="depth_sensor" type="air_pressure">
       <always_on>true</always_on>
-      <update_rate>50</update_rate>
+      <update_rate>100</update_rate>
       <air_pressure>
         <pressure>
