Commit message: added control package and modified com

File: src/atr_rov_description/urdf/atr_rov.urdf.xacro (robot description, xacro)
@@ -35,5 +35,6 @@
     <inertial>
       <!-- CoM offset — switches between display and physics frame -->
-      <origin xyz="-0.11 -0.001 ${com_z}" rpy="0 0 0"/>
+      <!-- <origin xyz="-0.11 -0.001 ${com_z}" rpy="0 0 0"/> -->
+      <origin xyz="0.06136 -0.00281 ${com_z}" rpy="0 0 0"/>
       <mass value="${mass}"/>
       <inertia ixx="${ixx}" ixy="${ixy}" ixz="${ixz}"
@@ -53,5 +54,6 @@
     </visual>
     <collision>
-      <origin xyz="-0.11 -0.001 0.22" rpy=" 0 0 0"/>
+      <!-- <origin xyz="-0.11 -0.001 0.22" rpy=" 0 0 0"/> -->
+      <origin xyz="0.06136 -0.001 0.22" rpy=" 0 0 0"/>
       <geometry>
         <box size="1.97 0.6 0.1038"/>
